File: sensors/dc_sensor_v2/dc_sensor_v2.sch (EAGLE design)
At the start: 22 parts, among them IC1 MCP602SN, IC2 MCP602SN, U1 IL300

Commit message: Updated DC voltage sensor to rev 2
Parts:
- added C10, C11, C9: (no value), resistor:C-EU025-040X050
- added C12, C15, C17, C20: (no value), resistor:C-EU025-030X050
- added C13, C14, C18, C19: (no value), resistor:C-EUC0603
- added C16, C21: (no value), resistor:CPOL-EUE2.5-6
- added IIN1, IIN2, VIN1: CTB1500/2, eko-parts:CTB1500/2
- added J1: F-1X04-SIP-100-40, con-headers-jp:F-1X04-SIP-100-40
- added J2: F-1X06-SIP-100-40, con-headers-jp:F-1X06-SIP-100-40
- added R11, R12, R13, R14, R15, R4: (no value), resistor:R-EU_0207/10
- added SJ1, SJ2: (no value), jumper:SJ
- added U$3, U$6: VRES_MURATA_PVZ2, eko-parts:VRES_MURATA_PVZ2
- added U2: IL300, ic-optoisolator:IL300
- added U3, U4: MCP601, eko-parts:MCP601
- added U5, U6: ACS712, eko-parts:ACS712
- C1, C2: device resistor:C-EU025-040X050 -> resistor:C-EUC1206
- C7: device resistor:C-EU025-040X050 -> resistor:CPOL-EUE2-5
- C8: device resistor:CPOL-EUE2-5 -> resistor:C-EU025-040X050
- U1: value IL300 -> MCE05S05S; device ic-optoisolator:IL300 -> modules:MCE05S05S
Connections:
- new net I_OUT1: C15.1, J2.4, R12.2
- new net I_OUT2: C20.1, J2.5, R15.2
- new net N$11: IIN1.1, U6.IP-3, U6.IP-4
- new net N$12: R10.2, SJ2.1, U$3.3
- new net N$13: C12.1, U6.FLT6
- new net N$14: R12.1, U3.VIN-, U3.VOUT
- new net N$15: IIN2.2, U5.IP+1, U5.IP+2
- new net N$16: R10.1, U6.VOUT7
- new net N$17: R11.2, SJ2.2, U$3.1, U$3.2, U3.VIN+
- new net N$18: IIN2.1, U5.IP-3, U5.IP-4
- new net N$19: C17.1, U5.FLT6
- new net N$20: R13.1, U5.VOUT7
- new net N$21: R14.2, SJ1.2, U$6.1, U$6.2, U4.VIN+
- new net N$22: R13.2, SJ1.1, U$6.3
- new net N$23: R15.1, U4.VIN-, U4.VOUT
- new net N$8: IC1A.+IN, R1.1, R4.2
- new net N$9: IIN1.2, U6.IP+1, U6.IP+2
- net +5V/1: now also C3.1, U1.VOUT+, U2.C_FB; no longer R6.2, U1.C_FB
- net +5V/2: now also C1.1, C13.1, C14.1, C16.+, C18.1, C19.1, C21.+, C6.1, C7.+, J1.3, R3.2, U1.VIN+, U2.C_OUT, U3.VDD, U4.VDD, U5.VCC8, U6.VCC8; no longer C7.1, C8.+, R10.2, U1.C_OUT
- net DC_OUT: now also C11.1, J2.1, R3.1, R5.2; no longer C6.1, R10.1, R9.2
- net DC_SENSE: now also R1.2, VIN1.2; no longer IC1A.+IN, R5.2, R6.1
- net GND1: now also C3.2, C8.1, R4.1, U1.VOUT-, U2.C_LED, VIN1.1; no longer R5.1, U1.C_LED
- net GND2: now also C1.2, C12.2, C13.2, C14.2, C15.2, C16.-, C17.2, C18.2, C19.2, C20.2, C21.-, C6.2, C7.-, J1.2, J1.4, J2.6, R11.1, R14.1, R9.1, U1.VIN-, U3.GND, U4.GND, U5.GND5, U6.GND5; no longer C7.2, C8.-, R3.1
- net N$1: now also C10.2, C9.2, R6.2, U2.A_FB; no longer C1.2, C3.2, R2.2, U1.A_FB
- net N$10: now also C11.2, R9.2; no longer C6.2, R7.2
- net N$2: now also R5.1; no longer R9.1
- net N$3: now also R7.2, U2.A_OUT; no longer R3.2, U1.A_OUT
- net N$4: now also C10.1, C8.2, R2.2, U2.A_LED; no longer C3.1, R1.2, U1.A_LED
- net N$5: now also C9.1, R2.1; no longer C1.1, R1.1
- net N$7: now also R6.1; no longer R2.1
Other:
- moved on the sheet: C1, C2, C3, C6, R1, R10, R2, R3, R5, R6, R7, R9
