File: Hardware/I_SenseTest/TEST1.brd (EAGLE design)
At the start: 57.1 x 39 mm, 18 parts

Commit message: Updated the Main Board
Main Board is Fully Done. need to Test the timing circuit before sending
the design for manufacture
Parts:
- C1: value (none) -> 1n
- C2: value (none) -> 100n
- R1, R2, R3, R6: value (none) -> 1k
- R4: value (none) -> 1.5k
- R5: value (none) -> 2k
Changed lines of the file:
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@@
 <element name="U$1" library="Pauls_parts" package="SOIC8" value="ACS712" x="12.7" y="19.05"/>
 <element name="U$2" library="Pauls_parts" package="PDIP8" value="MCP601" x="40.64" y="16.51" rot="R270"/>
-<element name="C1" library="resistor" package="C050-050X075" value="" x="11.43" y="5.08" rot="R180"/>
-<element name="C2" library="resistor" package="C050-050X075" value="" x="5.08" y="30.48" rot="R270"/>
-<element name="R1" library="resistor" package="0309/12" value="" x="24.13" y="5.08"/>
-<element name="R2" library="resistor" package="0309/12" value="" x="39.37" y="5.08"/>
-<element name="R3" library="resistor" package="0309/12" value="" x="25.4" y="19.05"/>
-<element name="R4" library="resistor" package="0309/12" value="" x="38.1" y="25.4"/>
+<element name="C1" library="resistor" package="C050-050X075" value="1n" x="11.43" y="5.08" rot="R180"/>
+<element name="C2" library="resistor" package="C050-050X075" value="100n" x="5.08" y="30.48" rot="R270"/>
+<element name="R1" library="resistor" package="0309/12" value="1k" x="24.13" y="5.08"/>
+<element name="R2" library="resistor" package="0309/12" value="1k" x="39.37" y="5.08"/>
+<element name="R3" library="resistor" package="0309/12" value="1k" x="25.4" y="19.05"/>
+<element name="R4" library="resistor" package="0309/12" value="1.5k" x="38.1" y="25.4"/>
 <element name="G2_OUT" library="testpad" package="P1-17Y" value="TPPAD1-17Y" x="44.45" y="33.02">
 <attribute name="TP_SIGNAL_NAME" value="" x="80.01" y="20.32" size="1.778" layer="27" display="off"/>
@@
 </element>
 <element name="U$3" library="Pauls_parts" package="PDIP8" value="MCP601" x="7.62" y="-5.08"/>
-<element name="R5" library="resistor" package="0309/12" value="" x="7.62" y="-21.59"/>
-<element name="R6" library="resistor" package="0309/12" value="" x="7.62" y="-27.94"/>
+<element name="R5" library="resistor" package="0309/12" value="2k" x="7.62" y="-21.59"/>
+<element name="R6" library="resistor" package="0309/12" value="1k" x="7.62" y="-27.94"/>
 <element name="G1_OUT" library="testpad" package="P1-17Y" value="TPPAD1-17Y" x="2.54" y="-13.97">
 <attribute name="TP_SIGNAL_NAME" value="" x="2.54" y="-34.29" size="1.778" layer="27" display="off"/>
