File: Hardware/Main Board/Main_Board_v2/Main_Board.sch (EAGLE design)
At the start: 49 parts, among them IC1 MBED_MICROCONTROLLER, IC2 NE555, Q1 IRF3704, Q2 BS170

Commit message: Main Board Ready for In-House Manufacture
Parts:
- added 2N7000: (no value), jumper:JP2E
- added U$4: INPUT_VOLTAGE_CONNECTOR, ekohub2013:INPUT_VOLTAGE_CONNECTOR
- C10: value (none) -> 10n
- DIS1: device display-lcd:TUXGR_16X2_R2 -> display-lcd3:TUXGR_16X2_R2
- JP10: value (none) -> POWER
- R13: value (none) -> 1M
- R4: value (none) -> 300k
- R7: value 60 -> 20
- renumbered POWER_SUPPLY to U$9
Connections:
- removed net BACKLIGHT: IC2.OUT, R7.1
- new net N$7: 2N7000.2, IC2.OUT
- new net P16_LCD: 2N7000.1, DIS1.NC@2
- net 5V_MBED: now also R7.1
- net GND: now also 2N7000.3; no longer DIS1.NC@2
- net VIN+: now also U$4.VIN+
- net VIN-: now also U$4.VIN-
Changed lines of the file:
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@@
 <setting verticaltext="up"/>
 </settings>
-<grid distance="0.1" unitdist="inch" unit="inch" style="lines" multiple="1" display="no" altdistance="0.01" altunitdist="inch" altunit="inch"/>
+<grid distance="0.1" unitdist="inch" unit="inch" style="lines" multiple="1" display="yes" altdistance="0.01" altunitdist="inch" altunit="inch"/>
 <layers>
 <layer number="1" name="Top" color="4" fill="1" visible="no" active="no"/>
@@
 <part name="U$3" library="Datalogging_Custom_Parts" deviceset="PANASONIC_CR2032" device=""/>
 <part name="JP9" library="jumper" deviceset="JP1E" device="" value="JP9"/>
-<part name="JP10" library="jumper" deviceset="JP1E" device=""/>
+<part name="JP10" library="jumper" deviceset="JP1E" device="" value="POWER"/>
 <part name="R6" library="rcl" deviceset="R-EU_" device="0411/12"/>
-<part name="R7" library="rcl" deviceset="R-EU_" device="0411/12" value="60"/>
+<part name="R7" library="rcl" deviceset="R-EU_" device="0411/12" value="20"/>
 <part name="D1" library="display-hp" deviceset="HLMP6" device=""/>
 <part name="R8" library="rcl" deviceset="R-EU_" device="0411/12"/>
@@
 <part name="Q1" library="transistor-power" deviceset="IRF3704" device=""/>
 <part name="Q2" library="transistor-small-signal" deviceset="BS170" device=""/>
-<part name="R13" library="rcl" deviceset="R-EU_" device="0411/12"/>
-<part name="POWER_SUPPLY" library="ekohub2013" deviceset="TRACO_ISOLATED_SUPPLY" device=""/>
+<part name="R13" library="rcl" deviceset="R-EU_" device="0411/12" value="1M"/>
 <part name="U$5" library="ekohub2013" deviceset="TACT_SWITCH" device=""/>
 <part name="R14" library="rcl" deviceset="R-EU_" device="0411/12" value="1K"/>
@@
 <part name="SUPPLY22" library="supply2" deviceset="GND" device=""/>
 <part name="SUPPLY23" library="supply2" deviceset="GND" device=""/>
-<part name="SUPPLY24" library="supply2" deviceset="GND" device=""/>
 <part name="SUPPLY25" library="supply2" deviceset="GND" device=""/>
 <part name="SUPPLY26" library="supply2" deviceset="GND" device=""/>
@@
 <part name="C9" library="capacitor-wima" deviceset="C" device="5/3" value="10uF"/>
 <part name="SUPPLY27" library="supply2" deviceset="GND" device=""/>
-<part name="DIS1" library="display-lcd" deviceset="TUXGR_16X2_R2" device=""/>
 <part name="IC2" library="st-microelectronics" deviceset="NE555" device=""/>
 <part name="C7" library="capacitor-wima" deviceset="C" device="5/3" value="10nF/0.01u"/>
 <part name="SUPPLY6" library="supply2" deviceset="GND" device=""/>
-<part name="C10" library="capacitor-wima" deviceset="C" device="5/3"/>
-<part name="R4" library="rcl" deviceset="R-EU_" device="0411/12"/>
+<part name="C10" library="capacitor-wima" deviceset="C" device="5/3" value="10n"/>
+<part name="R4" library="rcl" deviceset="R-EU_" device="0411/12" value="300k"/>
 <part name="SUPPLY7" library="supply2" deviceset="GND" device=""/>
+<part name="2N7000" library="jumper" deviceset="JP2E" device=""/>
+<part name="SUPPLY8" library="supply2" deviceset="GND" device=""/>
+<part name="U$9" library="ekohub2013" deviceset="TRACO_ISOLATED_SUPPLY" device=""/>
+<part name="U$4" library="ekohub2013" deviceset="INPUT_VOLTAGE_CONNECTOR" device=""/>
+<part name="DIS1" library="display-lcd3" deviceset="TUXGR_16X2_R2" device=""/>
 </parts>
 <sheets>
@@
 <instance part="Q2" gate="1" x="149.86" y="-26.67"/>
 <instance part="R13" gate="G$1" x="162.56" y="-13.97" rot="R90"/>
-<instance part="POWER_SUPPLY" gate="G$1" x="82.55" y="-55.88"/>
 <instance part="U$5" gate="G$1" x="189.23" y="-22.86" rot="R90"/>
 <instance part="R14" gate="G$1" x="217.17" y="-48.26" rot="R90"/>
@@
 <instance part="SUPPLY22" gate="GND" x="26.67" y="-60.96"/>
 <instance part="SUPPLY23" gate="GND" x="-8.89" y="-95.25"/>
-<instance part="SUPPLY24" gate="GND" x="-33.02" y="-77.47"/>
 <instance part="SUPPLY25" gate="GND" x="-73.66" y="-88.9"/>
 <instance part="SUPPLY26" gate="GND" x="105.41" y="-55.88"/>
@@
 <instance part="C9" gate="G$1" x="132.08" y="-54.61"/>
 <instance part="SUPPLY27" gate="GND" x="125.73" y="-67.31"/>
-<instance part="DIS1" gate="G$1" x="-55.88" y="-53.34"/>
 <instance part="IC2" gate="G$1" x="96.52" y="-106.68"/>
 <instance part="C7" gate="G$1" x="121.92" y="-116.84"/>
@@
 <instance part="R4" gate="G$1" x="66.04" y="-91.44" rot="R90"/>
 <instance part="SUPPLY7" gate="GND" x="66.04" y="-116.84"/>
+<instance part="2N7000" gate="1" x="147.32" y="-106.68" rot="R270"/>
+<instance part="SUPPLY8" gate="GND" x="142.24" y="-111.76"/>
+<instance part="U$9" gate="G$1" x="82.55" y="-55.88"/>
+<instance part="U$4" gate="G$1" x="175.26" y="-88.9"/>
+<instance part="DIS1" gate="G$1" x="-55.88" y="-53.34"/>
 </instances>
 <busses>
@@
 </segment>
 <segment>
-<pinref part="POWER_SUPPLY" gate="G$1" pin="VOUT-"/>
 <wire x1="97.79" y1="-53.34" x2="105.41" y2="-53.34" width="0.1524" layer="91"/>
 <label x="102.87" y="-52.07" size="1.4224" layer="95"/>
 <pinref part="SUPPLY26" gate="GND" pin="GND"/>
+<pinref part="U$9" gate="G$1" pin="VOUT-"/>
 </segment>
 <segment>
@@
 <wire x1="26.67" y1="-52.07" x2="26.67" y2="-58.42" width="0.1524" layer="91"/>
 <pinref part="SUPPLY22" gate="GND" pin="GND"/>
-</segment>
-<segment>
-<wire x1="-35.56" y1="-63.5" x2="-35.56" y2="-74.93" width="0.1524" layer="91"/>
-<wire x1="-35.56" y1="-74.93" x2="-33.02" y2="-74.93" width="0.1524" layer="91"/>
-<pinref part="SUPPLY24" gate="GND" pin="GND"/>
-<pinref part="DIS1" gate="G$1" pin="NC@2"/>
 </segment>
 <segment>
@@
 <wire x1="34.29" y1="-80.518" x2="34.29" y2="-83.82" width="0.1524" layer="91"/>
 </segment>
+<segment>
+<pinref part="2N7000" gate="1" pin="3"/>
+<pinref part="SUPPLY8" gate="GND" pin="GND"/>
+<wire x1="144.78" y1="-109.22" x2="142.24" y2="-109.22" width="0.1524" layer="91"/>
+</segment>
 </net>
 <net name="VIN" class="0">
@@
 </segment>
 <segment>
-<pinref part="POWER_SUPPLY" gate="G$1" pin="VOUT+"/>
 <label x="102.87" y="-46.99" size="1.4224" layer="95"/>
 <wire x1="97.79" y1="-48.26" x2="118.11" y2="-48.26" width="0.1524" layer="91"/>
@@
 <wire x1="132.08" y1="-52.07" x2="132.08" y2="-48.26" width="0.1524" layer="91"/>
 <junction x="132.08" y="-48.26"/>
+<pinref part="U$9" gate="G$1" pin="VOUT+"/>
 </segment>
 </net>
@@
 <wire x1="66.04" y1="-86.36" x2="66.04" y2="-83.82" width="0.1524" layer="91"/>
 <label x="66.802" y="-83.82" size="1.4224" layer="95"/>
+</segment>
+<segment>
+<pinref part="R7" gate="G$1" pin="1"/>
+<wire x1="-38.1" y1="-83.82" x2="-38.1" y2="-91.44" width="0.1524" layer="91"/>
+<label x="-35.56" y="-91.44" size="1.778" layer="95"/>
 </segment>
 </net>
@@
 <net name="VIN-" class="0">
 <segment>
-<pinref part="POWER_SUPPLY" gate="G$1" pin="VIN2-"/>
 <wire x1="67.31" y1="-53.34" x2="62.23" y2="-53.34" width="0.1524" layer="91"/>
 <wire x1="62.23" y1="-53.34" x2="62.23" y2="-50.8" width="0.1524" layer="91"/>
-<pinref part="POWER_SUPPLY" gate="G$1" pin="VIN1-"/>
 <wire x1="62.23" y1="-50.8" x2="62.23" y2="-48.26" width="0.1524" layer="91"/>
 <wire x1="62.23" y1="-48.26" x2="67.31" y2="-48.26" width="0.1524" layer="91"/>
@@
 <junction x="62.23" y="-50.8"/>
 <label x="54.61" y="-49.53" size="1.4224" layer="95"/>
+<pinref part="U$9" gate="G$1" pin="VIN1-"/>
+<pinref part="U$9" gate="G$1" pin="VIN2-"/>
+</segment>
+<segment>
+<wire x1="165.1" y1="-93.98" x2="152.4" y2="-93.98" width="0.1524" layer="91"/>
+<label x="152.4" y="-93.98" size="1.778" layer="95"/>
+<pinref part="U$4" gate="G$1" pin="VIN-"/>
 </segment>
 </net>
 <net name="VIN+" class="0">
 <segment>
-<pinref part="POWER_SUPPLY" gate="G$1" pin="VIN1+"/>
 <wire x1="67.31" y1="-58.42" x2="62.23" y2="-58.42" width="0.1524" layer="91"/>
 <wire x1="62.23" y1="-58.42" x2="62.23" y2="-60.96" width="0.1524" layer="91"/>
-<pinref part="POWER_SUPPLY" gate="G$1" pin="VIN2+"/>
 <wire x1="62.23" y1="-60.96" x2="62.23" y2="-63.5" width="0.1524" layer="91"/>
 <wire x1="67.31" y1="-63.5" x2="62.23" y2="-63.5" width="0.1524" layer="91"/>
@@
 <junction x="62.23" y="-60.96"/>
 <label x="54.61" y="-59.69" size="1.4224" layer="95"/>
+<pinref part="U$9" gate="G$1" pin="VIN1+"/>
+<pinref part="U$9" gate="G$1" pin="VIN2+"/>
+</segment>
+<segment>
+<wire x1="165.1" y1="-86.36" x2="152.4" y2="-86.36" width="0.1524" layer="91"/>
+<label x="152.4" y="-86.36" size="1.778" layer="95"/>
+<pinref part="U$4" gate="G$1" pin="VIN+"/>
 </segment>
 </net>
@@
 </segment>
 </net>
-<net name="BACKLIGHT" class="0">
-<segment>
-<pinref part="R7" gate="G$1" pin="1"/>
-<wire x1="-38.1" y1="-83.82" x2="-38.1" y2="-87.63" width="0.1524" layer="91"/>
-<label x="-35.56" y="-88.265" size="0.8128" layer="95" rot="R180"/>
-</segment>
-<segment>
-<pinref part="IC2" gate="G$1" pin="OUT"/>
-<wire x1="106.68" y1="-106.68" x2="121.92" y2="-106.68" width="0.1524" layer="91"/>
-<label x="114.3" y="-105.918" size="1.4224" layer="95"/>
-</segment>
-</net>
 <net name="N$2" class="0">
 <segment>
@@
 </segment>
 </net>
+<net name="N$7" class="0">
+<segment>
+<pinref part="IC2" gate="G$1" pin="OUT"/>
+<pinref part="2N7000" gate="1" pin="2"/>
+<wire x1="106.68" y1="-106.68" x2="144.78" y2="-106.68" width="0.1524" layer="91"/>
+</segment>
+</net>
+<net name="P16_LCD" class="0">
+<segment>
+<wire x1="-35.56" y1="-63.5" x2="-35.56" y2="-74.93" width="0.1524" layer="91"/>
+<wire x1="-35.56" y1="-74.93" x2="-30.48" y2="-74.93" width="0.1524" layer="91"/>
+<label x="-33.528" y="-77.724" size="1.778" layer="95"/>
+<pinref part="DIS1" gate="G$1" pin="NC@2"/>
+</segment>
+<segment>
+<pinref part="2N7000" gate="1" pin="1"/>
+<wire x1="144.78" y1="-104.14" x2="137.16" y2="-104.14" width="0.1524" layer="91"/>
+<label x="124.46" y="-104.14" size="1.778" layer="95"/>
+</segment>
+</net>

Commit message: Added Gerber Files for Main Board
Parts:
- removed Q1: IRF3704, transistor-power:IRF3704
- added Q3: IRF3704L-V, transistor-power:IRF3704L-V
Connections:
- net 5V: now also Q3.S; no longer Q1.S
- net MODEM: now also Q3.D; no longer Q1.D
- net N$5: now also Q3.G; no longer Q1.G
Changed lines of the file:
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@@
 <setting verticaltext="up"/>
 </settings>
-<grid distance="0.1" unitdist="inch" unit="inch" style="lines" multiple="1" display="yes" altdistance="0.01" altunitdist="inch" altunit="inch"/>
+<grid distance="0.1" unitdist="inch" unit="inch" style="lines" multiple="1" display="no" altdistance="0.01" altunitdist="inch" altunit="inch"/>
 <layers>
 <layer number="1" name="Top" color="4" fill="1" visible="no" active="no"/>
@@
 <part name="C2" library="capacitor-wima" deviceset="C" device="5/3" value="100nF"/>
 <part name="C3" library="capacitor-wima" deviceset="C" device="5/3" value="100nF"/>
-<part name="Q1" library="transistor-power" deviceset="IRF3704" device=""/>
 <part name="Q2" library="transistor-small-signal" deviceset="BS170" device=""/>
 <part name="R13" library="rcl" deviceset="R-EU_" device="0411/12" value="1M"/>
@@
 <part name="U$4" library="ekohub2013" deviceset="INPUT_VOLTAGE_CONNECTOR" device=""/>
 <part name="DIS1" library="display-lcd3" deviceset="TUXGR_16X2_R2" device=""/>
+<part name="Q3" library="transistor-power" deviceset="IRF3704" device="L-V"/>
 </parts>
 <sheets>
@@
 <instance part="C2" gate="G$1" x="-3.81" y="-83.82"/>
 <instance part="C3" gate="G$1" x="193.04" y="-46.99"/>
-<instance part="Q1" gate="G$1" x="149.86" y="-6.35" rot="R90"/>
 <instance part="Q2" gate="1" x="149.86" y="-26.67"/>
 <instance part="R13" gate="G$1" x="162.56" y="-13.97" rot="R90"/>
@@
 <instance part="U$4" gate="G$1" x="175.26" y="-88.9"/>
 <instance part="DIS1" gate="G$1" x="-55.88" y="-53.34"/>
+<instance part="Q3" gate="G$1" x="149.86" y="-6.35" rot="R90"/>
 </instances>
 <busses>
@@
 <net name="N$5" class="0">
 <segment>
-<pinref part="Q1" gate="G$1" pin="G"/>
 <pinref part="Q2" gate="1" pin="D"/>
 <wire x1="152.4" y1="-8.89" x2="152.4" y2="-20.32" width="0.1524" layer="91"/>
@@
 <wire x1="162.56" y1="-20.32" x2="152.4" y2="-20.32" width="0.1524" layer="91"/>
 <junction x="152.4" y="-20.32"/>
+<pinref part="Q3" gate="G$1" pin="G"/>
 </segment>
 </net>
 <net name="5V" class="0">
 <segment>
-<pinref part="Q1" gate="G$1" pin="S"/>
 <wire x1="154.94" y1="-3.81" x2="162.56" y2="-3.81" width="0.1524" layer="91"/>
 <pinref part="R13" gate="G$1" pin="2"/>
@@
 <junction x="162.56" y="-3.81"/>
 <label x="165.1" y="-1.27" size="1.4224" layer="95" rot="R180"/>
+<pinref part="Q3" gate="G$1" pin="S"/>
 </segment>
 </net>
 <net name="MODEM" class="0">
 <segment>
-<pinref part="Q1" gate="G$1" pin="D"/>
 <wire x1="144.78" y1="-3.81" x2="138.43" y2="-3.81" width="0.1524" layer="91"/>
 <label x="142.24" y="-1.27" size="1.4224" layer="95" rot="R180"/>
-</segment>
-<segment>
+<pinref part="Q3" gate="G$1" pin="D"/>
+</segment>
+<segment>

Commit message: Changed the TRACO Part and USB clearance fix
Changed lines of the file:
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@@
 <grid distance="0.1" unitdist="inch" unit="inch" style="lines" multiple="1" display="no" altdistance="0.01" altunitdist="inch" altunit="inch"/>
 <layers>
-<layer number="1" name="Top" color="4" fill="1" visible="no" active="no"/>
-<layer number="2" name="Route2" color="1" fill="3" visible="no" active="no"/>
-<layer number="3" name="Route3" color="4" fill="3" visible="no" active="no"/>
-<layer number="4" name="Route4" color="1" fill="4" visible="no" active="no"/>
-<layer number="5" name="Route5" color="4" fill="4" visible="no" active="no"/>
-<layer number="6" name="Route6" color="1" fill="8" visible="no" active="no"/>
-<layer number="7" name="Route7" color="4" fill="8" visible="no" active="no"/>
-<layer number="8" name="Route8" color="1" fill="2" visible="no" active="no"/>
-<layer number="9" name="Route9" color="4" fill="2" visible="no" active="no"/>
-<layer number="10" name="Route10" color="1" fill="7" visible="no" active="no"/>
-<layer number="11" name="Route11" color="4" fill="7" visible="no" active="no"/>
-<layer number="12" name="Route12" color="1" fill="5" visible="no" active="no"/>
-<layer number="13" name="Route13" color="4" fill="5" visible="no" active="no"/>
-<layer number="14" name="Route14" color="1" fill="6" visible="no" active="no"/>
-<layer number="15" name="Route15" color="4" fill="6" visible="no" active="no"/>
-<layer number="16" name="Bottom" color="1" fill="1" visible="no" active="no"/>
-<layer number="17" name="Pads" color="2" fill="1" visible="no" active="no"/>
-<layer number="18" name="Vias" color="2" fill="1" visible="no" active="no"/>
-<layer number="19" name="Unrouted" color="6" fill="1" visible="no" active="no"/>
-<layer number="20" name="Dimension" color="15" fill="1" visible="no" active="no"/>
-<layer number="21" name="tPlace" color="7" fill="1" visible="no" active="no"/>
-<layer number="22" name="bPlace" color="7" fill="1" visible="no" active="no"/>
-<layer number="23" name="tOrigins" color="15" fill="1" visible="no" active="no"/>
-<layer number="24" name="bOrigins" color="15" fill="1" visible="no" active="no"/>
-<layer number="25" name="tNames" color="7" fill="1" visible="no" active="no"/>
-<layer number="26" name="bNames" color="7" fill="1" visible="no" active="no"/>
-<layer number="27" name="tValues" color="7" fill="1" visible="no" active="no"/>
-<layer number="28" name="bValues" color="7" fill="1" visible="no" active="no"/>
+<layer number="1" name="Top" color="4" fill="1" visible="yes" active="no"/>
+<layer number="2" name="Route2" color="1" fill="3" visible="yes" active="no"/>
+<layer number="3" name="Route3" color="4" fill="3" visible="yes" active="no"/>
+<layer number="4" name="Route4" color="1" fill="4" visible="yes" active="no"/>
+<layer number="5" name="Route5" color="4" fill="4" visible="yes" active="no"/>
+<layer number="6" name="Route6" color="1" fill="8" visible="yes" active="no"/>
+<layer number="7" name="Route7" color="4" fill="8" visible="yes" active="no"/>
+<layer number="8" name="Route8" color="1" fill="2" visible="yes" active="no"/>
+<layer number="9" name="Route9" color="4" fill="2" visible="yes" active="no"/>
+<layer number="10" name="Route10" color="1" fill="7" visible="yes" active="no"/>
+<layer number="11" name="Route11" color="4" fill="7" visible="yes" active="no"/>
+<layer number="12" name="Route12" color="1" fill="5" visible="yes" active="no"/>
+<layer number="13" name="Route13" color="4" fill="5" visible="yes" active="no"/>
+<layer number="14" name="Route14" color="1" fill="6" visible="yes" active="no"/>
+<layer number="15" name="Route15" color="4" fill="6" visible="yes" active="no"/>
+<layer number="16" name="Bottom" color="1" fill="1" visible="yes" active="no"/>
+<layer number="17" name="Pads" color="2" fill="1" visible="yes" active="no"/>
+<layer number="18" name="Vias" color="2" fill="1" visible="yes" active="no"/>
+<layer number="19" name="Unrouted" color="6" fill="1" visible="yes" active="no"/>
+<layer number="20" name="Dimension" color="15" fill="1" visible="yes" active="no"/>
+<layer number="21" name="tPlace" color="7" fill="1" visible="yes" active="no"/>
+<layer number="22" name="bPlace" color="7" fill="1" visible="yes" active="no"/>
+<layer number="23" name="tOrigins" color="15" fill="1" visible="yes" active="no"/>
+<layer number="24" name="bOrigins" color="15" fill="1" visible="yes" active="no"/>
+<layer number="25" name="tNames" color="7" fill="1" visible="yes" active="no"/>
+<layer number="26" name="bNames" color="7" fill="1" visible="yes" active="no"/>
+<layer number="27" name="tValues" color="7" fill="1" visible="yes" active="no"/>
+<layer number="28" name="bValues" color="7" fill="1" visible="yes" active="no"/>
 <layer number="29" name="tStop" color="7" fill="3" visible="no" active="no"/>
 <layer number="30" name="bStop" color="7" fill="6" visible="no" active="no"/>
@@
 <layer number="35" name="tGlue" color="7" fill="4" visible="no" active="no"/>
 <layer number="36" name="bGlue" color="7" fill="5" visible="no" active="no"/>
-<layer number="37" name="tTest" color="7" fill="1" visible="no" active="no"/>
-<layer number="38" name="bTest" color="7" fill="1" visible="no" active="no"/>
+<layer number="37" name="tTest" color="7" fill="1" visible="yes" active="no"/>
+<layer number="38" name="bTest" color="7" fill="1" visible="yes" active="no"/>
 <layer number="39" name="tKeepout" color="4" fill="11" visible="no" active="no"/>
 <layer number="40" name="bKeepout" color="1" fill="11" visible="no" active="no"/>
@@
 <layer number="44" name="Drills" color="7" fill="1" visible="no" active="no"/>
 <layer number="45" name="Holes" color="7" fill="1" visible="no" active="no"/>
-<layer number="46" name="Milling" color="3" fill="1" visible="no" active="no"/>
-<layer number="47" name="Measures" color="7" fill="1" visible="no" active="no"/>
-<layer number="48" name="Document" color="7" fill="1" visible="no" active="no"/>
-<layer number="49" name="Reference" color="7" fill="1" visible="no" active="no"/>
-<layer number="50" name="dxf" color="7" fill="1" visible="no" active="no"/>
-<layer number="51" name="tDocu" color="7" fill="1" visible="no" active="no"/>
-<layer number="52" name="bDocu" color="7" fill="1" visible="no" active="no"/>
-<layer number="53" name="tGND_GNDA" color="7" fill="1" visible="no" active="no"/>
-<layer number="54" name="bGND_GNDA" color="7" fill="1" visible="no" active="no"/>
-<layer number="56" name="wert" color="7" fill="1" visible="no" active="no"/>
+<layer number="46" name="Milling" color="3" fill="1" visible="yes" active="no"/>
+<layer number="47" name="Measures" color="7" fill="1" visible="yes" active="no"/>
+<layer number="48" name="Document" color="7" fill="1" visible="yes" active="no"/>
+<layer number="49" name="Reference" color="7" fill="1" visible="yes" active="no"/>
+<layer number="50" name="dxf" color="7" fill="1" visible="yes" active="no"/>
+<layer number="51" name="tDocu" color="7" fill="1" visible="yes" active="no"/>
+<layer number="52" name="bDocu" color="7" fill="1" visible="yes" active="no"/>
+<layer number="53" name="tGND_GNDA" color="7" fill="1" visible="yes" active="no"/>
+<layer number="54" name="bGND_GNDA" color="7" fill="1" visible="yes" active="no"/>
+<layer number="56" name="wert" color="7" fill="1" visible="yes" active="no"/>
 <layer number="91" name="Nets" color="2" fill="1" visible="yes" active="yes"/>
 <layer number="92" name="Busses" color="1" fill="1" visible="yes" active="yes"/>
