File: Hardware/Main Board/Main_Board_v3/Main_Board.brd (EAGLE design)
At the start: 105.4 x 84.8 mm, 68 parts, among them IC1 MBED_MICROCONTROLLER, IC2 NE555, Q1 BS170, Q2 BS170, Q3 IRF3704L-V, Q4 IRF3704L-V, Q5 BS170, Q6 IRF3704L-V, Q7 BS170, Q8 IRF3704L-V

Commit message: Added Reverse Polarity Protection
Parts:
- added D6: 1N4148DO35-10, diode:DO35-10
- moved R13 1.27 mm to (74.9, 76.2)
- moved R10 1.27 mm to (99.1, 10.9)
Connections:
- net VIN+: now also D6.A
- net VIN-: now also D6.C
Routing:
- net VIN-: track 43.6 -> 70.7 mm
- net GND: track 20.8 -> 11.0 mm
- net VIN+: track 22.9 -> 29.2 mm
- net N$5: track 26.9 -> 29.5 mm
- net N$15: track 13.5 -> 14.7 mm
Changed lines of the file:
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@@
 <layer number="27" name="tValues" color="7" fill="1" visible="yes" active="yes"/>
 <layer number="28" name="bValues" color="7" fill="1" visible="yes" active="yes"/>
-<layer number="29" name="tStop" color="7" fill="3" visible="no" active="yes"/>
-<layer number="30" name="bStop" color="7" fill="6" visible="no" active="yes"/>
-<layer number="31" name="tCream" color="7" fill="4" visible="no" active="yes"/>
-<layer number="32" name="bCream" color="7" fill="5" visible="no" active="yes"/>
-<layer number="33" name="tFinish" color="6" fill="3" visible="no" active="yes"/>
-<layer number="34" name="bFinish" color="6" fill="6" visible="no" active="yes"/>
-<layer number="35" name="tGlue" color="7" fill="4" visible="no" active="yes"/>
-<layer number="36" name="bGlue" color="7" fill="5" visible="no" active="yes"/>
-<layer number="37" name="tTest" color="7" fill="1" visible="no" active="yes"/>
-<layer number="38" name="bTest" color="7" fill="1" visible="no" active="yes"/>
+<layer number="29" name="tStop" color="7" fill="3" visible="yes" active="yes"/>
+<layer number="30" name="bStop" color="7" fill="6" visible="yes" active="yes"/>
+<layer number="31" name="tCream" color="7" fill="4" visible="yes" active="yes"/>
+<layer number="32" name="bCream" color="7" fill="5" visible="yes" active="yes"/>
+<layer number="33" name="tFinish" color="6" fill="3" visible="yes" active="yes"/>
+<layer number="34" name="bFinish" color="6" fill="6" visible="yes" active="yes"/>
+<layer number="35" name="tGlue" color="7" fill="4" visible="yes" active="yes"/>
+<layer number="36" name="bGlue" color="7" fill="5" visible="yes" active="yes"/>
+<layer number="37" name="tTest" color="7" fill="1" visible="yes" active="yes"/>
+<layer number="38" name="bTest" color="7" fill="1" visible="yes" active="yes"/>
 <layer number="39" name="tKeepout" color="4" fill="11" visible="yes" active="yes"/>
 <layer number="40" name="bKeepout" color="1" fill="11" visible="yes" active="yes"/>
@@
 <layer number="42" name="bRestrict" color="1" fill="10" visible="yes" active="yes"/>
 <layer number="43" name="vRestrict" color="2" fill="10" visible="yes" active="yes"/>
-<layer number="44" name="Drills" color="7" fill="1" visible="no" active="yes"/>
-<layer number="45" name="Holes" color="7" fill="1" visible="no" active="yes"/>
-<layer number="46" name="Milling" color="3" fill="1" visible="no" active="yes"/>
-<layer number="47" name="Measures" color="7" fill="1" visible="no" active="yes"/>
+<layer number="44" name="Drills" color="7" fill="1" visible="yes" active="yes"/>
+<layer number="45" name="Holes" color="7" fill="1" visible="yes" active="yes"/>
+<layer number="46" name="Milling" color="3" fill="1" visible="yes" active="yes"/>
+<layer number="47" name="Measures" color="7" fill="1" visible="yes" active="yes"/>
 <layer number="48" name="Document" color="7" fill="1" visible="yes" active="yes"/>
 <layer number="49" name="Reference" color="7" fill="1" visible="yes" active="yes"/>
@@
 <layer number="250" name="Descript" color="7" fill="1" visible="yes" active="yes"/>
 <layer number="251" name="SMDround" color="7" fill="1" visible="yes" active="yes"/>
-<layer number="254" name="cooling" color="7" fill="1" visible="no" active="yes"/>
+<layer number="254" name="cooling" color="7" fill="1" visible="yes" active="yes"/>
 </layers>
 <board>
@@
 <param name="rvMicroViaOuter" value="0.25"/>
 <param name="rvMicroViaInner" value="0.25"/>
-<param name="rlMinPadTop" value="20mil"/>
+<param name="rlMinPadTop" value="14mil"/>
 <param name="rlMaxPadTop" value="25mil"/>
-<param name="rlMinPadInner" value="10mil"/>
+<param name="rlMinPadInner" value="14mil"/>
 <param name="rlMaxPadInner" value="20mil"/>
-<param name="rlMinPadBottom" value="20mil"/>
+<param name="rlMinPadBottom" value="14mil"/>
 <param name="rlMaxPadBottom" value="25mil"/>
 <param name="rlMinViaOuter" value="20mil"/>
@@
 <element name="R2" library="rcl" package="0411/12" value="" x="59.182" y="52.07" rot="R90"/>
 <element name="R3" library="rcl" package="0411/12" value="" x="64.516" y="52.07" rot="R90"/>
-<element name="U$1" library="ekohub2013" package="USBA_SOCKET" value="USBA_SOCKET" x="55.88" y="72.39" rot="R180"/>
+<element name="U$1" library="ekohub2013" package="USBA_SOCKET" value="USBA_SOCKET" x="55.88" y="72.39" smashed="yes" rot="R180"/>
 <element name="D1" library="display-hp" package="HLMP6" value="HLMP6" x="89.662" y="15.875" rot="R270">
 <attribute name="OC_NEWARK" value="40K0088" x="-39.878" y="-8.255" size="1.778" layer="27" rot="R270" display="off"/>
@@
 <attribute name="OC_FARNELL" value="1652490" x="-47.117" y="-36.195" size="1.778" layer="27" rot="R270" display="off"/>
 </element>
-<element name="R10" library="rcl" package="0411/12" value="" x="97.79" y="10.922" rot="R180"/>
+<element name="R10" library="rcl" package="0411/12" value="" x="99.06" y="10.922" rot="R180"/>
 <element name="D4" library="display-hp" package="HLMP6" value="HLMP6" x="78.613" y="15.875" rot="R270">
 <attribute name="OC_NEWARK" value="40K0088" x="-50.927" y="-50.165" size="1.778" layer="27" rot="R270" display="off"/>
@@
 <element name="C3" library="capacitor-wima" package="C5B3.5" value="100nF" x="30.48" y="26.67" rot="R90"/>
 <element name="Q2" library="transistor-small-signal" package="SOT54E" value="BS170" x="67.31" y="70.866" rot="R90"/>
-<element name="R13" library="rcl" package="0411/12" value="1M" x="73.66" y="76.2" rot="R270"/>
+<element name="R13" library="rcl" package="0411/12" value="1M" x="74.93" y="76.2" rot="R270"/>
 <element name="U$5" library="ekohub2013" package="TACT_SWITCH" value="TACT_SWITCH" x="34.036" y="17.272"/>
 <element name="R14" library="rcl" package="0411/12" value="1K" x="47.117" y="29.21" rot="R270"/>
@@
 <element name="R20" library="rcl" package="0411/12" value="1M" x="10.8458" y="20.3962" rot="R90"/>
 <element name="Q8" library="transistor-power" package="TO262-V" value="IRF3704L-V" x="5.7658" y="21.59" rot="R90"/>
+<element name="D6" library="diode" package="DO35-10" value="1N4148DO35-10" x="6.35" y="68.58" rot="R270"/>
 </elements>
 <signals>
@@
 </polygon>
 <wire x1="67.31" y1="72.136" x2="67.31" y2="72.39" width="0.6096" layer="16"/>
-<wire x1="58.03" y1="72.39" x2="58.03" y2="71.86" width="0.6096" layer="16"/>
 <contactref element="JP15" pad="2"/>
 <contactref element="JP16" pad="2"/>
@@
 <via x="100.33" y="66.548" extent="1-16" drill="0.8" shape="square"/>
 <wire x1="100.33" y1="66.548" x2="100.33" y2="63.5" width="0.4064" layer="16"/>
-<wire x1="58.03" y1="72.39" x2="67.31" y2="72.39" width="0.4064" layer="16"/>
 <contactref element="Q5" pad="S"/>
 <contactref element="C11" pad="1"/>
@@
 <wire x1="82.423" y1="14.605" x2="82.042" y2="14.605" width="0.4064" layer="16"/>
 <wire x1="82.042" y1="14.605" x2="82.042" y2="10.922" width="0.4064" layer="16"/>
-<wire x1="82.042" y1="10.922" x2="91.44" y2="10.922" width="0.4064" layer="16"/>
+<wire x1="82.042" y1="10.922" x2="92.71" y2="10.922" width="0.4064" layer="16"/>
 </signal>
 <signal name="N$16">
@@
 <contactref element="Q3" pad="1"/>
 <contactref element="R13" pad="1"/>
-<wire x1="67.31" y1="81.28" x2="73.66" y2="81.28" width="0.6096" layer="16"/>
-<wire x1="73.66" y1="81.28" x2="73.66" y2="82.55" width="0.6096" layer="16"/>
-<wire x1="70.358" y1="80.01" x2="73.66" y2="80.01" width="0.6096" layer="1"/>
-<wire x1="73.66" y1="80.01" x2="73.66" y2="82.55" width="0.6096" layer="1"/>
-<wire x1="70.358" y1="80.01" x2="70.358" y2="69.596" width="0.6096" layer="1"/>
-<wire x1="70.358" y1="69.596" x2="67.31" y2="69.596" width="0.6096" layer="1"/>
+<wire x1="67.31" y1="81.28" x2="74.93" y2="81.28" width="0.6096" layer="16"/>
+<wire x1="74.93" y1="81.28" x2="74.93" y2="82.55" width="0.6096" layer="16"/>
+<wire x1="71.628" y1="80.01" x2="74.93" y2="80.01" width="0.6096" layer="1"/>
+<wire x1="74.93" y1="80.01" x2="74.93" y2="82.55" width="0.6096" layer="1"/>
+<wire x1="71.628" y1="80.01" x2="71.628" y2="69.596" width="0.6096" layer="1"/>
+<wire x1="71.628" y1="69.596" x2="67.31" y2="69.596" width="0.6096" layer="1"/>
 </signal>
 <signal name="MODEM">
@@
 <wire x1="20.066" y1="66.04" x2="22.01" y2="66.04" width="1.4224" layer="16"/>
 <wire x1="22.01" y1="66.04" x2="22.01" y2="69.85" width="1.4224" layer="16"/>
+<contactref element="D6" pad="C"/>
+<wire x1="6.35" y1="73.66" x2="11.43" y2="73.66" width="1.016" layer="1"/>
+<wire x1="11.43" y1="73.66" x2="11.43" y2="66.04" width="1.016" layer="1"/>
+<wire x1="11.43" y1="66.04" x2="22.01" y2="66.04" width="1.016" layer="1"/>
+<wire x1="22.01" y1="66.04" x2="22.01" y2="69.85" width="1.016" layer="1"/>
 </signal>
 <signal name="VIN+">
@@
 <wire x1="7.62" y1="58.42" x2="16.51" y2="58.42" width="1.4224" layer="16"/>
 <wire x1="16.51" y1="58.42" x2="16.51" y2="69.85" width="1.4224" layer="16"/>
+<contactref element="D6" pad="A"/>
+<wire x1="6.35" y1="63.5" x2="7.62" y2="63.5" width="1.016" layer="16"/>
+<wire x1="7.62" y1="63.5" x2="7.62" y2="58.42" width="1.016" layer="16"/>
 </signal>
 <signal name="N$2">
@@
 <wire x1="16.51" y1="10.16" x2="7.62" y2="10.16" width="0.4064" layer="1"/>
 <wire x1="7.62" y1="10.16" x2="7.62" y2="12.7" width="0.4064" layer="1"/>
-<wire x1="7.62" y1="12.7" x2="7.4676" y2="12.7" width="0" layer="19" extent="1-1"/>
+<wire x1="7.62" y1="12.7" x2="7.4676" y2="12.7" width="0.254" layer="1"/>
 </signal>
 </signals>

Commit message: Board Layouts done for DC Current and AC Board
Changed lines of the file:
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@@
 <wire x1="62.23" y1="53.34" x2="35.4584" y2="53.3908" width="0.4064" layer="1"/>
 <wire x1="35.4584" y1="53.3908" x2="35.4584" y2="74.4982" width="0.4064" layer="1"/>
-<wire x1="35.4584" y1="74.4982" x2="19.7358" y2="74.4474" width="0.4064" layer="1"/>
-<wire x1="19.7358" y1="74.4474" x2="19.7358" y2="74.9808" width="0.4064" layer="1"/>
-<wire x1="19.7358" y1="74.9808" x2="19.685" y2="74.93" width="0" layer="19" extent="1-1"/>
+<wire x1="35.4584" y1="74.4982" x2="19.685" y2="74.4982" width="0.4064" layer="1"/>
+<wire x1="19.685" y1="74.4982" x2="19.685" y2="74.93" width="0.4064" layer="1"/>
 </signal>
 <signal name="N$7">
