File: Hardware/Sensor Boards/DCCurrent/DCCurrentV1/DCCurrent.brd (EAGLE design)
At the start: 160 x 100 mm, 43 parts, among them IC1 MCP604P, IC2 MCP604P, U7 AD7993BRUZ-0

Commit message: Board Layouts done for DC Current and AC Board
Parts:
- removed C1, C10, C2, C9: 1n, resistor:C050-050X075
- removed C12, C13, C14: (no value), ee2parts:E2,5-7---100UF
- added C11, C15, C16, C17, C6, C7, C8: (no value), resistor:E2-4
- added U$10, U$12, U$7, U$8: (no value), holes:3,0
- C3, C4, C5: device ee2parts:E2,5-7---100UF -> resistor:E2-4
- moved C25 142.3 mm to (58.4, 49.5)
- moved R38 119.6 mm to (50.8, 63.5), turned to 180 degrees
- moved R24 112.5 mm to (34.3, 31.8), turned to 180 degrees
- moved R37 103.9 mm to (50.8, 67.3), turned to 180 degrees
- moved R18 103.8 mm to (34.3, 49.5), turned to 180 degrees
- moved R6 101.3 mm to (34.3, 77.5), turned to 180 degrees
- moved R10 100.8 mm to (34.3, 59.7), turned to 180 degrees
- moved R17 100.4 mm to (47.0, 53.3), turned to 90 degrees
- moved R21 97.2 mm to (34.3, 35.6)
- moved R26 95.3 mm to (34.3, 24.1), turned to 180 degrees
- moved R1 90.1 mm to (34.3, 88.9)
- moved R16 89.3 mm to (50.8, 53.3), turned to 270 degrees
- moved R5 86.9 mm to (34.3, 81.3)
- moved R9 85.3 mm to (34.3, 63.5)
- moved R25 81.8 mm to (34.3, 27.9)
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Connections:
- net +5V: now also C15.+, C16.+, C17.+, C6.+, C8.+; no longer C12.+, C13.+, C14.+, C4.+, C5.+
- net GND: now also C11.-, C15.-, C16.-, C17.-, C6.-, C7.-, C8.-; no longer C1.2, C10.2, C12.-, C13.-, C14.-, C2.2, C9.2
- net N$12: now also C5.+; no longer C2.1
- net N$22: now also C7.+; no longer C9.1
- net N$31: now also C11.+; no longer C10.1
- net N$5: now also C4.+; no longer C1.1
Routing:
- added copper zone on layer 16, net GND
Other:
- board size 160 x 100 mm -> 63.5 x 77.1 mm
