File: Hardware/Sensor Boards/DCCurrent/DCCurrentV2/DCCurrent.brd (EAGLE design)
At the start: 97.5 x 80 mm, 53 parts, among them IC1 MCP604P, IC2 MCP604P, U1 IL300, U10 IL300, U13 AD7993BRUZ-0, U5 IL300, U7 IL300

Commit message: DC Current Board - Done by Saurab
Parts:
- removed C1, C18, C2, C26, C28, C30: (no value), resistor:C025-040X050
- removed C29, C31: (no value), resistor:E2-5
- removed C35: (no value), resistor:C025-025X050
- removed JP3: (no value), jumper:JP4
- removed R11, R12, R13, R14, R2, R22, R3: (no value), resistor:0207/10
- removed U1, U10, U5: IL300, ic-optoisolator:DIL08
- removed U13: AD7993BRUZ-0, ADC:SOP65P640X120-16N
- added C11, C15, C16, C6, C7, C8: (no value), resistor:E2-4
- added R24, R37, R38: 1.5k, resistor:0309/12
- added R25: 2k, resistor:0309/12
- added R26: 1k, resistor:0309/12
- added U$10, U$12: (no value), holes:3,0
- added U$11, U$9: ACS712, Pauls_parts:SOIC8
- C17, C25, C3, C4: device resistor:C025-040X050 -> resistor:E2-4
- JP1: device jumper:JP4 -> connectors:JP4
- R1, R10, R15, R16, R17, R20, R21, R6, R7: value (none) -> 1k; device resistor:0207/10 -> resistor:0309/12
- R18, R4, R8: value (none) -> 1.5k; device resistor:0207/10 -> resistor:0309/12
- R19, R5, R9: value (none) -> 2k; device resistor:0207/10 -> resistor:0309/12
- U$1, U$4: value (none) -> ACS712; device holes:3,0 -> Pauls_parts:SOIC8
- U$2, U$3: value (none) -> INPUT_VOLTAGE_CONNECTOR; device holes:3,0 -> ekohub2013:INPUT_VOLTAGE_CONNECTOR
- U$7, U$8: value INPUT_VOLTAGE_CONNECTOR -> (none); device ekohub2013:INPUT_VOLTAGE_CONNECTOR -> holes:3,0
- U7: value IL300 -> AD7993BRUZ-0; device ic-optoisolator:DIL08 -> ADC:SOP65P640X120-16N
- moved C5 249.8 mm to (23.5, 53.3), turned to 270 degrees
- moved C4 248.5 mm to (23.5, 69.2), turned to 270 degrees
- moved C3 247.3 mm to (24.8, 74.3), turned to 90 degrees
- moved U7 181.7 mm to (57.1, 55.9), turned to 90 degrees
- moved IC2 178.9 mm to (49.5, 80.0), turned to 270 degrees
- moved U$7 145.1 mm to (3.81, 92.7)
- moved C25 138.4 mm to (61.0, 45.7)
- moved U$6 118.7 mm to (14.0, 82.5)
- moved U$3 91.4 mm to (14.0, 49.5)
- moved U$8 90.7 mm to (3.81, 22.2)
- moved U$2 90.1 mm to (14.0, 33.0)
- moved U$5 86.4 mm to (14.0, 66.0)
- moved U$1 70.9 mm to (17.8, 73.7), turned to 270 degrees
- moved R5 59.3 mm to (36.2, 82.5), turned to 0 degrees
- moved IC1 53.4 mm to (48.3, 31.8), turned to 90 degrees
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Connections:
- removed net +5V/1: C28.1, C29.+, IC1.4, JP3.3, U1.3, U10.3, U5.3, U7.3
- removed net +5V/2: C30.1, C31.+, C35.1, C5.+, IC2.4, JP1.1, R21.1, R22.1, U1.6, U10.6, U13.5, U13.6, U5.6, U7.6
- removed net DC_OUT1: IC2.1, IC2.2, U13.7
- removed net DC_OUT2: IC2.6, IC2.7, U13.10
- removed net DC_OUT3: IC2.8, IC2.9, U13.8
- removed net DC_OUT4: IC2.13, IC2.14, U13.9
- removed net DC_SENSE1: R1.2, U$8.V+
- removed net DC_SENSE2: R10.2, U$7.V+
- removed net DC_SENSE3: R15.2, U$6.V+
- removed net DC_SENSE4: R20.2, U$5.V+
- removed net GND1: C28.2, C29.-, IC1.11, IC1.13, JP3.4, R12.1, R14.1, R17.1, R19.1, R4.1, R5.1, R6.1, R9.1, U$5.V-, U$6.V-, U$7.V-, U$8.V-, U1.1, U5.1, U7.1
- removed net GND2: C30.2, C31.-, C35.2, C5.-, IC2.11, JP1.2, R13.1, R18.1, R7.1, R8.1, U10.1, U13.1, U13.11, U13.16, U13.2, U13.3, U13.4
- removed net N$17: C26.1, R16.2, U10.2
- removed net N$18: C25.1, IC1.1, R16.1
- removed net N$23: C17.2, C18.2, IC1.6, R12.2, U7.4
- new net +5V: C15.+, C16.+, C17.+, C25.+, C3.+, C6.+, C8.+, IC1.4, IC2.4, JP1.1, R16.2, R37.1, R38.1, U$1.8, U$11.8, U$4.8, U$9.8, U7.11, U7.5, U7.6
- new net 2.5V: IC1.10, IC1.12, IC1.3, IC1.5, IC2.10, IC2.12, IC2.3, IC2.5, R16.1, R17.2
- new net GND: C11.-, C15.-, C16.-, C17.-, C25.-, C3.-, C4.-, C5.-, C6.-, C7.-, C8.-, IC1.11, IC2.11, JP1.2, R17.1, U$1.5, U$11.5, U$4.5, U$9.5, U7.1, U7.16, U7.2, U7.3, U7.4
- new net N$11: IC2.9, R7.2, R8.1
- new net N$22: C7.+, U$9.6
- new net N$25: IC1.6, R19.2, R20.1
- new net N$26: IC1.1, R18.2, R19.1
- new net N$27: U$11.3, U$11.4, U$2.V+
- new net N$28: U$11.1, U$11.2, U$2.V-
- new net N$29: R21.1, U$11.7
- new net N$30: IC1.9, R21.2, R24.1
- new net N$31: C11.+, U$11.6
- new net N$33: IC1.8, R24.2, R25.1
- new net N$34: IC1.13, R25.2, R26.1
- new net VAC_OUT1: IC1.7, R20.2, U7.7
- new net VAC_OUT2: IC1.14, R26.2, U7.10
- new net VAC_OUT3: IC2.14, R10.2, U7.9
- new net VAC_OUT4: IC2.7, R6.2, U7.8
- net N$1: now also U$1.3, U$1.4, U$6.V+; no longer C3.2, C4.2, R6.2, U1.4
- net N$10: now also R7.1, U$4.7; no longer IC1.10, R10.1, R9.2
- net N$12: now also C5.+, U$4.6; no longer C18.1, R11.2, U7.2
- net N$13: now also IC2.8, R8.2, R9.1; no longer C17.1, IC1.7, R11.1
- net N$14: now also U$3.V+, U$9.3, U$9.4; no longer IC2.5, R13.2, U7.5
- net N$15: now also IC2.13, R10.1, R9.2; no longer IC1.5, R14.2, R15.1
- net N$16: now also U$3.V-, U$9.1, U$9.2; no longer C25.2, C26.2, IC1.2, R17.2, U10.4
- net N$19: now also R15.1, U$9.7; no longer IC2.3, R18.2, U10.5
- net N$2: now also U$1.1, U$1.2, U$6.V-; no longer C1.2, C2.2, IC1.9, R5.2, U5.4
- net N$20: now also IC1.2, R15.2, R18.1; no longer IC1.3, R19.2, R20.1
- net N$3: now also R1.1, U$1.7; no longer IC2.12, R7.2, U1.5
- net N$4: now also IC2.2, R1.2, R4.1; no longer C4.1, R2.2, U1.2
- net N$5: now also C4.+, U$1.6; no longer C3.1, IC1.14, R2.1
- net N$6: now also IC2.1, R4.2, R5.1; no longer C1.1, R3.2, U5.2
- net N$7: now also IC2.6, R5.2, R6.1; no longer C2.1, IC1.8, R3.1
- net N$8: now also U$4.3, U$4.4, U$5.V+; no longer IC1.12, R1.1, R4.2
- net N$9: now also U$4.1, U$4.2, U$5.V-; no longer IC2.10, R8.2, U5.5
- net SCL: now also R37.2, U7.15; no longer R22.2, U13.15
- net SDA: now also R38.2, U7.14; no longer R21.2, U13.14
Routing:
- net +5V: track 0.00 -> 285.5 mm, vias 0 -> 2
- net 2.5V: track 0.00 -> 101.1 mm
- net VAC_OUT3: track 0.00 -> 94.4 mm
- net N$15: track 0.00 -> 81.1 mm
- net VAC_OUT4: track 0.00 -> 76.9 mm
- net GND: track 0.00 -> 72.7 mm
- net N$20: track 0.00 -> 71.3 mm
- net N$26: track 0.00 -> 63.9 mm
- net VAC_OUT2: track 0.00 -> 62.0 mm
- net VAC_OUT1: track 0.00 -> 57.5 mm
- net N$25: track 0.00 -> 34.4 mm
- net N$11: track 0.00 -> 29.6 mm
- net N$13: track 0.00 -> 29.1 mm
- net N$33: track 0.00 -> 28.6 mm
- net SDA: track 0.00 -> 23.9 mm
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- added copper zone on layer 1, net GND
- added copper zone on layer 16, net GND
- removed copper zone on layer 1, net GND1
- removed copper zone on layer 1, net GND2
- removed copper zone on layer 1, net PE
Other:
- board size 97.5 x 80 mm -> 64.8 x 77.8 mm
- board text removed: "+5V/1"
- board text removed: "+5V/2"
- board text removed: "DC Voltage"
- board text removed: "GND1"
- board text removed: "GND2"
- board text removed: "SCL"
- board text removed: "SDA"
- board text removed: "ekoHUB v2"
