File: Hardware/Sensor Boards/DCCurrent/DCCurrentV2/DCCurrent.sch (EAGLE design)
At the start: 63 parts, among them IC1 MCP604P, IC2 MCP604P, U1 IL300, U10 IL300, U13 AD7993BRUZ-0, U2 MCP602-E/P, U3 MCP602-E/P, U4 IL300, U5 MCP602-E/P, U6 MCP602-E/P, U7 IL300

Commit message: DC Current Board - Done by Saurab
Parts:
- removed C1, C10, C14, C18, C26, C28, C30, C9: (no value), resistor:C-EU025-040X050
- removed C29, C31: (no value), resistor:CPOL-EUE2-5
- removed C33: (no value), resistor:C-EU025-024X044
- removed C34: (no value), resistor:CPOL-EUE2-4
- removed C35: (no value), resistor:C-EU025-025X050
- removed JP3: (no value), jumper:JP4E
- removed R11, R12, R13, R14, R2, R22, R3: (no value), resistor:R-EU_0207/10
- removed U$7, U$8: INPUT_VOLTAGE_CONNECTOR, ekohub2013:INPUT_VOLTAGE_CONNECTOR
- removed U1, U10, U4: IL300, ic-optoisolator:IL300
- removed U13: AD7993BRUZ-0, ADC:AD7993BRUZ-0
- removed U2, U3, U5, U6: MCP602-E/P, MCP:MCP602-E/P
- added R24, R37, R38: 1.5k, resistor:R-EU_0309/12
- added R25: 2k, resistor:R-EU_0309/12
- added R26: 1k, resistor:R-EU_0309/12
- added U$1, U$11, U$4, U$9: ACS712, Pauls_parts:ACS712
- added U$2, U$3: INPUT_VOLTAGE_CONNECTOR, ekohub2013:INPUT_VOLTAGE_CONNECTOR
- C11, C16, C17, C25, C3, C5, C6, C8: device resistor:C-EU025-040X050 -> resistor:CPOL-EUE2-4
- C15, C4, C7: device resistor:CPOL-EUE2-5 -> resistor:CPOL-EUE2-4
- JP1: device jumper:JP4E -> connectors:JP4E
- R1, R10, R15, R16, R17, R20, R21, R6, R7: value (none) -> 1k; device resistor:R-EU_0207/10 -> resistor:R-EU_0309/12
- R18, R4, R8: value (none) -> 1.5k; device resistor:R-EU_0207/10 -> resistor:R-EU_0309/12
- R19, R5, R9: value (none) -> 2k; device resistor:R-EU_0207/10 -> resistor:R-EU_0309/12
- U7: value IL300 -> AD7993BRUZ-0; device ic-optoisolator:IL300 -> ADC:AD7993BRUZ-0
Connections:
- removed net +5V/1: C28.1, C29.+, C3.1, C4.+, C5.1, IC1P.V+, JP3.3, U1.C_FB, U10.C_FB, U2.VDD, U4.C_FB, U7.C_FB
- removed net +5V/2: C14.1, C15.+, C30.1, C31.+, C33.1, C34.+, C35.1, C6.1, C7.+, IC2P.V+, JP1.3, R21.1, R22.1, U1.C_OUT, U10.C_OUT, U13.AS, U13.REFIN, U13.VDD, U3.VDD, U4.C_OUT, U6.VDD, U7.C_OUT
- removed net DC_OUT1: IC2A.-IN, IC2A.OUT, U13.VIN1
- removed net DC_OUT2: IC2B.-IN, IC2B.OUT, U13.VIN2
- removed net DC_OUT3: U13.VIN3, U6.VINA-, U6.VOUTA
- removed net DC_OUT4: U13.VIN4, U3.VINA-, U3.VOUTA
- removed net DC_SENSE1: R1.2, U$8.VIN+
- removed net DC_SENSE2: R10.2, U$7.VIN+
- removed net DC_SENSE3: R15.2, U$6.VIN+
- removed net DC_SENSE4: R20.2, U$5.VIN+
- removed net GND1: C16.1, C28.2, C29.-, C3.2, C4.-, C5.2, C8.1, IC1P.V-, JP3.4, R12.1, R14.1, R17.1, R19.1, R4.1, R5.1, R6.1, R9.1, U$5.VIN-, U$6.VIN-, U$7.VIN-, U$8.VIN-, U1.C_LED, U2.VINB+, U2.VSS, U4.C_LED, U5.VINB+, U5.VSS, U7.C_LED
- removed net GND2: C14.2, C15.-, C30.2, C31.-, C33.2, C34.-, C35.2, C6.2, C7.-, IC2P.V-, JP1.4, R13.1, R18.1, R7.1, R8.1, U10.C_LED, U13.AGND, U13.AGND_2, U13.AGND_3, U13.AGND_4, U13.AGND_5, U3.VINB+, U3.VSS, U6.VINB+, U6.VSS
- removed net N$17: C26.1, R16.2, U10.A_LED
- removed net N$18: C25.1, IC1A.OUT, R16.1
- removed net N$21: JP1.1, R21.2, U13.SDA
- removed net N$23: C17.2, C18.2, IC1B.-IN, R12.2, U7.A_FB
- removed net N$32: U5.VOUTB
- removed net N$36: U2.VINB-, U2.VOUTB
- removed net N$38: U3.VINB-, U3.VOUTB
- new net +5V: C15.+, C16.+, C17.+, C25.+, C3.+, C6.+, C8.+, IC1P.V+, IC2P.V+, JP1.1, R16.2, R37.1, R38.1, U$1.VCC8, U$11.VCC8, U$4.VCC8, U$9.VCC8, U7.AS, U7.REFIN, U7.VDD
- new net 2.5V: IC1A.+IN, IC1B.+IN, IC1C.+IN, IC1D.+IN, IC2A.+IN, IC2B.+IN, IC2C.+IN, IC2D.+IN, R16.1, R17.2
- new net GND: C11.-, C15.-, C16.-, C17.-, C25.-, C3.-, C4.-, C5.-, C6.-, C7.-, C8.-, IC1P.V-, IC2P.V-, JP1.2, R17.1, U$1.GND5, U$11.GND5, U$4.GND5, U$9.GND5, U7.AGND, U7.AGND_2, U7.AGND_3, U7.AGND_4, U7.AGND_5
- new net N$11: IC2C.-IN, R7.2, R8.1
- new net N$25: IC1B.-IN, R19.2, R20.1
- new net N$26: IC1A.OUT, R18.2, R19.1
- new net N$27: U$11.IP-3, U$11.IP-4, U$2.VIN+
- new net N$28: U$11.IP+1, U$11.IP+2, U$2.VIN-
- new net N$29: R21.1, U$11.VOUT7
- new net N$30: IC1C.-IN, R21.2, R24.1
- new net N$31: C11.+, U$11.FLT6
- new net N$33: IC1C.OUT, R24.2, R25.1
- new net SCL: JP1.4, R37.2, U7.SCL
- new net SDA: JP1.3, R38.2, U7.SDA
- new net VAC_OUT1: IC1B.OUT, R20.2, U7.VIN1
- new net VAC_OUT2: IC1D.OUT, R26.2, U7.VIN2
- new net VAC_OUT3: IC2D.OUT, R10.2, U7.VIN4
- new net VAC_OUT4: IC2B.OUT, R6.2, U7.VIN3
- net N$1: now also U$1.IP-3, U$1.IP-4, U$6.VIN+; no longer C10.2, C9.2, R6.2, U1.A_FB, U2.VINA-
- net N$10: now also R7.1, U$4.VOUT7; no longer R10.1, R9.2, U5.VINA+
- net N$12: now also C5.+, U$4.FLT6; no longer C18.1, R11.2, U7.A_LED
- net N$13: now also IC2C.OUT, R8.2, R9.1; no longer C17.1, IC1B.OUT, R11.1
- net N$14: now also U$3.VIN+, U$9.IP-3, U$9.IP-4; no longer IC2B.+IN, R13.2, U7.A_OUT
- net N$15: now also IC2D.-IN, R10.1, R9.2; no longer IC1B.+IN, R14.2, R15.1
- net N$16: now also U$3.VIN-, U$9.IP+1, U$9.IP+2; no longer C25.2, C26.2, IC1A.-IN, R17.2, U10.A_FB
- net N$19: now also R15.1, U$9.VOUT7; no longer IC2A.+IN, R18.2, U10.A_OUT
- net N$2: now also U$1.IP+1, U$1.IP+2, U$6.VIN-; no longer C1.2, C11.2, R5.2, U4.A_FB
- net N$20: now also IC1A.-IN, R15.2, R18.1; no longer IC1A.+IN, R19.2, R20.1
- net N$22: now also C7.+, U$9.FLT6; no longer JP1.2, R22.2, U13.SCL
- net N$3: now also R1.1, U$1.VOUT7; no longer R7.2, U1.A_OUT, U3.VINA+
- net N$34: now also IC1D.-IN, R25.2, R26.1; no longer U6.VINB-, U6.VOUTB
- net N$4: now also IC2A.-IN, R1.2, R4.1; no longer C10.1, C8.2, R2.2, U1.A_LED
- net N$5: now also C4.+, U$1.FLT6; no longer C9.1, R2.1, U2.VOUTA
- net N$6: now also IC2A.OUT, R4.2, R5.1; no longer C11.1, C16.2, R3.2, U4.A_LED
- net N$7: now also IC2B.-IN, R5.2, R6.1; no longer C1.1, R3.1, U5.VOUTA
- net N$8: now also U$4.IP-3, U$4.IP-4, U$5.VIN+; no longer R1.1, R4.2, U2.VINA+
- net N$9: now also U$4.IP+1, U$4.IP+2, U$5.VIN-; no longer R8.2, U4.A_OUT, U6.VINA+
Other:
- moved on the sheet: C15, C4, C7, IC1A, IC1B, IC1C, IC1D, IC2A, IC2B, IC2C, IC2D, JP1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
