File: Hardware/Sensor Boards/DCVoltage/DCVoltageV1/VDC.brd (EAGLE design)
At the start: 67 x 80 mm, 53 parts, among them IC1 MCP604P, IC2 MCP604P, U1 IL300, U10 IL300, U13 AD7993BRUZ-0, U5 IL300, U7 IL300

Commit message: DC Current Board - Done by Saurab
Parts:
- removed R13, R18, R7, R8: (no value), resistor:0207/10
- added R23, R24, R25, R26: (no value), rcl:IRG2014TRIM
- moved C17 34.1 mm to (38.1, 27.3)
- moved C18 34.1 mm to (38.1, 21.0)
- moved C25 32.6 mm to (38.1, 14.6)
- moved C26 32.3 mm to (38.1, 8.89)
- moved C29 31.1 mm to (19.7, 40.0), turned to 0 degrees
- moved C2 31.1 mm to (37.5, 61.0), turned to 270 degrees
- moved C28 31.1 mm to (19.7, 34.9), turned to 0 degrees
- moved C1 31.0 mm to (37.5, 54.6), turned to 90 degrees
- moved R3 30.9 mm to (47.0, 53.3)
- moved R9 30.9 mm to (47.0, 58.4)
- moved C30 30.5 mm to (5.08, 27.3)
- moved JP1 30.5 mm to (13.7, 4.14)
- moved R11 30.5 mm to (47.6, 36.2)
- moved R12 30.5 mm to (47.6, 38.7)
- moved R14 30.5 mm to (47.6, 41.3)
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Connections:
- net GND1: now also U10.1
- net GND2: now also R23.P$1, R23.P$2, R24.P$1, R24.P$2, R25.P$1, R25.P$2, R26.P$1, R26.P$2; no longer R13.1, R18.1, R7.1, R8.1, U10.1
- net N$14: now also R24.P$3; no longer R13.2
- net N$19: now also R23.P$3; no longer R18.2
- net N$3: now also R26.P$3; no longer R7.2
- net N$9: now also R25.P$3; no longer R8.2
Routing:
- net +5V/2: track 0.00 -> 79.5 mm
- net +5V/1: track 0.00 -> 66.3 mm
- net N$7: track 0.00 -> 27.3 mm
- net N$5: track 0.00 -> 26.0 mm
- net N$23: track 0.00 -> 15.2 mm
- net N$1: track 0.00 -> 15.2 mm
- net N$2: track 0.00 -> 14.6 mm
- net DC_SENSE2: track 0.00 -> 12.7 mm
- net N$4: track 0.00 -> 12.1 mm
- net N$6: track 0.00 -> 11.4 mm
- net DC_SENSE1: track 0.00 -> 10.8 mm
- net N$3: track 0.00 -> 7.40 mm
- net N$9: track 0.00 -> 4.45 mm
- net N$14: track 0.00 -> 3.81 mm
- net N$16: track 0.00 -> 3.18 mm
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