File: Hardware/Sensor Boards/DCVoltage/DCVoltageV1/VDC.sch (EAGLE design)
At the start: 43 parts, among them IC1 MCP604P, IC2 MCP604P, U7 AD7993BRUZ-0

Commit message: DC Voltage Sensor board added
Parts:
- removed C11, C15, C16, C6, C7, C8: (no value), resistor:CPOL-EUE2-4
- removed R24, R37, R38: 1.5k, resistor:R-EU_0309/12
- removed R25: 2k, resistor:R-EU_0309/12
- removed R26: 1k, resistor:R-EU_0309/12
- removed U$1, U$11, U$4, U$9: ACS712, Pauls_parts:ACS712
- removed U$2, U$3: INPUT_VOLTAGE_CONNECTOR, ekohub2013:INPUT_VOLTAGE_CONNECTOR
- added C1, C18, C2, C26, C28, C30: (no value), resistor:C-EU025-040X050
- added C29, C31: (no value), resistor:CPOL-EUE2-5
- added C35: (no value), resistor:C-EU025-025X050
- added JP3: (no value), jumper:JP4E
- added R11, R12, R13, R14, R2, R22, R3: (no value), resistor:R-EU_0207/10
- added U$7, U$8: INPUT_VOLTAGE_CONNECTOR, ekohub2013:INPUT_VOLTAGE_CONNECTOR
- added U1, U10, U5: IL300, ic-optoisolator:IL300
- added U13: AD7993BRUZ-0, ADC:AD7993BRUZ-0
- C17, C25, C3, C4: device resistor:CPOL-EUE2-4 -> resistor:C-EU025-040X050
- JP1: device connectors:JP4E -> jumper:JP4E
- R1, R10, R15, R16, R17, R20, R21, R6, R7: value 1k -> (none); device resistor:R-EU_0309/12 -> resistor:R-EU_0207/10
- R18, R4, R8: value 1.5k -> (none); device resistor:R-EU_0309/12 -> resistor:R-EU_0207/10
- R19, R5, R9: value 2k -> (none); device resistor:R-EU_0309/12 -> resistor:R-EU_0207/10
- U7: value AD7993BRUZ-0 -> IL300; device ADC:AD7993BRUZ-0 -> ic-optoisolator:IL300
Connections:
- removed net +5V: C15.+, C16.+, C17.+, C25.+, C3.+, C6.+, C8.+, IC1P.V+, IC2P.V+, JP1.1, R16.2, R37.1, R38.1, U$1.VCC8, U$11.VCC8, U$4.VCC8, U$9.VCC8, U7.AS, U7.REFIN, U7.VDD
- removed net 2.5V: IC1A.+IN, IC1B.+IN, IC1C.+IN, IC1D.+IN, IC2A.+IN, IC2B.+IN, IC2C.+IN, IC2D.+IN, R16.1, R17.2
- removed net GND: C11.-, C15.-, C16.-, C17.-, C25.-, C3.-, C4.-, C5.-, C6.-, C7.-, C8.-, IC1P.V-, IC2P.V-, JP1.2, R17.1, U$1.GND5, U$11.GND5, U$4.GND5, U$9.GND5, U7.AGND, U7.AGND_2, U7.AGND_3, U7.AGND_4, U7.AGND_5
- removed net N$11: IC2C.-IN, R7.2, R8.1
- removed net N$22: C7.+, U$9.FLT6
- removed net N$25: IC1B.-IN, R19.2, R20.1
- removed net N$26: IC1A.OUT, R18.2, R19.1
- removed net N$27: U$11.IP-3, U$11.IP-4, U$2.VIN+
- removed net N$28: U$11.IP+1, U$11.IP+2, U$2.VIN-
- removed net N$29: R21.1, U$11.VOUT7
- removed net N$30: IC1C.-IN, R21.2, R24.1
- removed net N$31: C11.+, U$11.FLT6
- removed net N$33: IC1C.OUT, R24.2, R25.1
- removed net N$34: IC1D.-IN, R25.2, R26.1
- removed net VAC_OUT1: IC1B.OUT, R20.2, U7.VIN1
- removed net VAC_OUT2: IC1D.OUT, R26.2, U7.VIN2
- removed net VAC_OUT3: IC2D.OUT, R10.2, U7.VIN4
- removed net VAC_OUT4: IC2B.OUT, R6.2, U7.VIN3
- new net +5V/1: C28.1, C29.+, IC1P.V+, JP3.3, U1.C_FB, U10.C_FB, U5.C_FB, U7.C_FB
- new net +5V/2: C30.1, C31.+, C35.1, C5.+, IC2P.V+, JP1.1, R21.1, R22.1, U1.C_OUT, U10.C_OUT, U13.REFIN, U13.VDD, U5.C_OUT, U7.C_OUT
- new net DC_OUT1: IC2A.-IN, IC2A.OUT, U13.VIN1
- new net DC_OUT2: IC2B.-IN, IC2B.OUT, U13.VIN2
- new net DC_OUT3: IC2C.-IN, IC2C.OUT, U13.VIN3
- new net DC_OUT4: IC2D.-IN, IC2D.OUT, U13.VIN4
- new net DC_SENSE1: R1.2, U$8.VIN+
- new net DC_SENSE2: R10.2, U$7.VIN+
- new net DC_SENSE3: R15.2, U$6.VIN+
- new net DC_SENSE4: R20.2, U$5.VIN+
- new net GND1: C28.2, C29.-, IC1D.-IN, IC1P.V-, JP3.4, R12.1, R14.1, R17.1, R19.1, R4.1, R5.1, R6.1, R9.1, U$5.VIN-, U$6.VIN-, U$7.VIN-, U$8.VIN-, U1.C_LED, U5.C_LED, U7.C_LED
- new net GND2: C30.2, C31.-, C35.2, C5.-, IC2P.V-, JP1.2, R13.1, R18.1, R7.1, R8.1, U10.C_LED, U13.AGND, U13.AGND_2, U13.AGND_3, U13.AGND_4, U13.AGND_5, U13.AS
- new net N$17: C26.1, R16.2, U10.A_LED
- new net N$18: C25.1, IC1A.OUT, R16.1
- new net N$23: C17.2, C18.2, IC1B.-IN, R12.2, U7.A_FB
- net N$1: now also C3.2, C4.2, R6.2, U1.A_FB; no longer U$1.IP-3, U$1.IP-4, U$6.VIN+
- net N$10: now also IC1C.+IN, R10.1, R9.2; no longer R7.1, U$4.VOUT7
- net N$12: now also C18.1, R11.2, U7.A_LED; no longer C5.+, U$4.FLT6
- net N$13: now also C17.1, IC1B.OUT, R11.1; no longer IC2C.OUT, R8.2, R9.1
- net N$14: now also IC2B.+IN, R13.2, U7.A_OUT; no longer U$3.VIN+, U$9.IP-3, U$9.IP-4
- net N$15: now also IC1B.+IN, R14.2, R15.1; no longer IC2D.-IN, R10.1, R9.2
- net N$16: now also C25.2, C26.2, IC1A.-IN, R17.2, U10.A_FB; no longer U$3.VIN-, U$9.IP+1, U$9.IP+2
- net N$19: now also IC2A.+IN, R18.2, U10.A_OUT; no longer R15.1, U$9.VOUT7
- net N$2: now also C1.2, C2.2, IC1C.-IN, R5.2, U5.A_FB; no longer U$1.IP+1, U$1.IP+2, U$6.VIN-
- net N$20: now also IC1A.+IN, R19.2, R20.1; no longer IC1A.-IN, R15.2, R18.1
- net N$3: now also IC2D.+IN, R7.2, U1.A_OUT; no longer R1.1, U$1.VOUT7
- net N$4: now also C4.1, R2.2, U1.A_LED; no longer IC2A.-IN, R1.2, R4.1
- net N$5: now also C3.1, IC1D.OUT, R2.1; no longer C4.+, U$1.FLT6
- net N$6: now also C1.1, R3.2, U5.A_LED; no longer IC2A.OUT, R4.2, R5.1
- net N$7: now also C2.1, IC1C.OUT, R3.1; no longer IC2B.-IN, R5.2, R6.1
- net N$8: now also IC1D.+IN, R1.1, R4.2; no longer U$4.IP-3, U$4.IP-4, U$5.VIN+
- net N$9: now also IC2C.+IN, R8.2, U5.A_OUT; no longer U$4.IP+1, U$4.IP+2, U$5.VIN-
- net SCL: now also R22.2, U13.SCL; no longer R37.2, U7.SCL
- net SDA: now also R21.2, U13.SDA; no longer R38.2, U7.SDA
Other:
- moved on the sheet: C5, IC1A, IC1B, IC1C, IC1D, IC2A, IC2B, IC2C, IC2D, JP1, R1, R10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

Commit message: DC Current Board - Done by Saurab
Parts:
- removed R13, R18, R7, R8: (no value), resistor:R-EU_0207/10
- added R23, R24, R25, R26: (no value), rcl:R-TRIMM
Connections:
- net GND1: now also U10.C_LED
- net GND2: now also R23.A, R23.S, R24.A, R24.S, R25.A, R25.S, R26.A, R26.S; no longer R13.1, R18.1, R7.1, R8.1, U10.C_LED
- net N$14: now also R24.E; no longer R13.2
- net N$19: now also R23.E; no longer R18.2
- net N$3: now also R26.E; no longer R7.2
- net N$9: now also R25.E; no longer R8.2
